File: relControll.kicad_pcb (KiCad board)
At the start: 2 copper layers, 196.2 x 67.3 mm, 40 parts, among them J1 left side, J2 right side, J3 Conn_01x06_Socket, J4 Conn_01x06_Socket, SW1 PEC11R-4015F-S0024, U1 74HC4051, U2 74HC4051, U3 6N137S_C20612601

Commit message: fix
Parts:
- removed R13, R14: 10kΩ, PCM_JLCPCB:R_0805
- added H1: MountingHole, MountingHole:MountingHole_2.7mm_M2.5_ISO14580_Pad, F.Cu at (152.7, 62.2)
- added N1: Housing, Symbol:Screw_Generic_2.0x3.0mm_SilkScreen, F.Cu at (157.3, 61.9)
- MIDI1, MIDI2: footprint EasyEDA:AUDIO-SMD_PJ-327E-5A -> EasyEDA:AUDIO-TH_PJ-3270
- R15: footprint PCM_JLCPCB:R_0805 -> EasyEDA:R0805
- moved R15 4.30 mm to (99.0, 99.8)
- turned MIDI1 to 180 degrees
- turned MIDI2 to 180 degrees
Connections:
- MIDI1 pad 3: opto_src -> /sleeve
- MIDI1 pad 5: SENS -> opto_src
- MIDI2 pad 3: /ring2 -> GND
- MIDI2 pad 5: SENS2 -> /ring2
- R15 pad 2: Net-(R14-Pad2) -> SW
- SW1 pad 2: Net-(R14-Pad2) -> SW
- SW1 pad 3: (no net) -> GND
- SW1 pad 4: (no net) -> GND
Routing:
- net Net-(R13-Pad2): track 21.4 -> 0.00 mm
- net Net-(R14-Pad2): track 20.7 -> 0.00 mm, vias 1 -> 0
- net SW: track 5.84 -> 24.5 mm, vias 0 -> 1
- net VCC: track 464.6 -> 473.3 mm
- net A: track 46.8 -> 41.1 mm
- net opto_src: track 14.6 -> 10.7 mm
- net GND: track 2.99 -> 0.01 mm, vias 93 -> 99
- net /sleeve: track 10.5 -> 8.67 mm
- net B: track 53.4 -> 51.7 mm
- net /ring2: track 8.23 -> 6.86 mm
- net VDD: track 443.1 -> 442.2 mm
- net /tip2: track 14.3 -> 13.4 mm
- net Rx: track 29.5 -> 28.9 mm
