File: relControll.kicad_sch (KiCad schematic)
At the start: 38 parts, among them J1 left side, J2 right side, J3 Conn_01x06_Socket, J4 Conn_01x06_Socket, SW1 PEC11R-4015F-S0024, U1 74HC4051, U2 74HC4051, U3 6N137S_C20612601

Commit message: fix
Parts:
- removed R14: 10kΩ, PCM_JLCPCB:R_0805, symbol -- JLCPCB --:0805,10kΩ
- added H1: MountingHole, MountingHole:MountingHole_2.7mm_M2.5_ISO14580_Pad, symbol Mechanical:MountingHole
- added N1: Housing, Symbol:Screw_Generic_2.0x3.0mm_SilkScreen, symbol Mechanical:Housing
- MIDI1, MIDI2: footprint EasyEDA:AUDIO-SMD_PJ-327E-5A -> EasyEDA:AUDIO-TH_PJ-3270; symbol EasyEDA:PJ-327E-5A -> EasyEDA:PJ-3270; LCSC Part C145812 -> C381134; MPN PJ-327E-5A -> PJ-3270; Manufacturer 韩国韩荣 -> XKB Connection(中国星坤)
- R15: footprint PCM_JLCPCB:R_0805 -> EasyEDA:R0805
Connections:
- net GND: now also MIDI2.3, SW1.3 (MT1), SW1.4 (MT2); no longer MIDI2.1, SW1.MT1, SW1.MT2
- net SENS: now also MIDI1.6; no longer MIDI1.5
- net SENS2: now also MIDI2.6; no longer MIDI2.5
- net SW: now also R15.2, SW1.2
- net opto_src: now also MIDI1.5; no longer MIDI1.3
- net ring2: now also MIDI2.5; no longer MIDI2.3
- net sleeve: now also MIDI1.3; no longer MIDI1.1
Other:
- moved on the sheet: SW1
